File: hardware/BREAD_Slice.kicad_pcb (KiCad board)
At the start: 2 copper layers, 70 x 100 mm, 16 parts, among them J1 I2C_01x04, J2 Conn_01x10_Female

Commit message: completed board
Parts:
- added BT1: Battery_Cell, Battery:BatteryHolder_Keystone_3000_1x12mm, F.Cu at (167.9, 46.5)
- added BZ1: CX-1612C, Buzzer_Beeper:Buzzer_15x7.5RM7.6, F.Cu at (128.8, 60.9)
- added C10: 0.1u, Capacitor_SMD:C_1206_3216Metric_Pad1.33x1.80mm_HandSolder, B.Cu at (145.6, 56.3)
- added C11: 1.0u, Capacitor_SMD:C_1206_3216Metric_Pad1.33x1.80mm_HandSolder, B.Cu at (143.2, 51.3)
- added C12: 1.0u, Capacitor_SMD:C_1206_3216Metric_Pad1.33x1.80mm_HandSolder, B.Cu at (143.2, 56.3)
- added C13: 22p, Capacitor_SMD:C_1206_3216Metric_Pad1.33x1.80mm_HandSolder, B.Cu at (167.2, 45.1)
- added C14: 1u, Capacitor_SMD:C_1206_3216Metric_Pad1.33x1.80mm_HandSolder, B.Cu at (141.9, 92.7)
- added C15: 1u, Capacitor_SMD:C_1206_3216Metric_Pad1.33x1.80mm_HandSolder, B.Cu at (149.9, 91.4)
- added C5: 0.1uF, Capacitor_SMD:C_0805_2012Metric, F.Cu at (171.2, 109.3)
- added C6: 0.1uF, Capacitor_SMD:C_0805_2012Metric, F.Cu at (171.2, 112.1)
- added C7: 0.1u, Capacitor_SMD:C_1206_3216Metric_Pad1.33x1.80mm_HandSolder, F.Cu at (171.5, 87.0)
- added C8: 10u, Capacitor_SMD:C_1206_3216Metric_Pad1.33x1.80mm_HandSolder, F.Cu at (169.1, 87.0)
- added C9: 0.1u, Capacitor_SMD:C_1206_3216Metric_Pad1.33x1.80mm_HandSolder, B.Cu at (145.6, 51.3)
- added D2: H178CAD, KML-Custom:H178CAD_P2.54mm_RightAngle_LED, F.Cu at (135.5, 45.6)
- added D3: 1N4007, Diode_THT:D_DO-35_SOD27_P7.62mm_Horizontal, F.Cu at (136.4, 51.7)
- added D4: 1N4148, Diode_THT:D_DO-35_SOD27_P7.62mm_Horizontal, F.Cu at (168.7, 62.5)
- added IC1: DS3234S#, KML-Custom:SOIC127P1032X265-20N, B.Cu at (168.4, 54.8)
- added J3: MicroSD_502570-0893, KML-Custom:MicroSD_5025700893, F.Cu at (149.4, 49.0)
- added JP1: Jumper_3_Bridged12, Jumper:SolderJumper-3_P1.3mm_Bridged2Bar12_Pad1.0x1.5mm_NumberLabels, F.Cu at (161.9, 110.0)
- added JP2: Jumper_3_Bridged12, Jumper:SolderJumper-3_P1.3mm_Bridged2Bar12_Pad1.0x1.5mm_NumberLabels, F.Cu at (161.9, 112.6)
- added JP3: Jumper_2_Open, Jumper:SolderJumper-2_P1.3mm_Open_TrianglePad1.0x1.5mm, F.Cu at (169.6, 104.1)
- added K2: SANYOU_SRD_Form_C, Relay_THT:Relay_SPDT_SANYOU_SRD_Series_Form_C, F.Cu at (167.1, 65.7)
- added PR1: 4.7k, Resistor_SMD:R_1206_3216Metric_Pad1.30x1.75mm_HandSolder, F.Cu at (165.7, 104.8)
- added PR2: 4.7k, Resistor_SMD:R_1206_3216Metric_Pad1.30x1.75mm_HandSolder, F.Cu at (161.9, 106.1)
- added PR3: 4.7k, Resistor_SMD:R_1206_3216Metric_Pad1.30x1.75mm_HandSolder, F.Cu at (161.8, 116.8)
- added PR4: 4.7k, Resistor_SMD:R_1206_3216Metric_Pad1.30x1.75mm_HandSolder, F.Cu at (167.3, 110.0)
- added Q1: IRLZ34N, Package_TO_SOT_THT:TO-220-3_Horizontal_TabDown, F.Cu at (143.9, 69.2)
- added Q2: IRLZ34N, Package_TO_SOT_THT:TO-220-3_Horizontal_TabDown, F.Cu at (156.3, 65.4)
- added R1: 85, Resistor_SMD:R_1206_3216Metric_Pad1.30x1.75mm_HandSolder, B.Cu at (136.0, 48.7)
- added R10: 10K, Resistor_SMD:R_1206_3216Metric_Pad1.30x1.75mm_HandSolder, F.Cu at (171.4, 90.8)
- added R11: 100k, Resistor_SMD:R_1206_3216Metric_Pad1.30x1.75mm_HandSolder, B.Cu at (144.5, 47.7)
- added R12: 100k, Resistor_SMD:R_1206_3216Metric_Pad1.30x1.75mm_HandSolder, B.Cu at (140.9, 47.2)
- added R13: 100k, Resistor_SMD:R_1206_3216Metric_Pad1.30x1.75mm_HandSolder, B.Cu at (155.8, 47.3)
- added R14: 100k, Resistor_SMD:R_1206_3216Metric_Pad1.30x1.75mm_HandSolder, B.Cu at (145.6, 60.0)
- added R15: 10k, Resistor_SMD:R_1206_3216Metric_Pad1.30x1.75mm_HandSolder, B.Cu at (167.2, 47.6)
- added R16: 10K, Resistor_SMD:R_1206_3216Metric_Pad1.30x1.75mm_HandSolder, B.Cu at (141.9, 90.2)
- added R2: 220, Resistor_SMD:R_1206_3216Metric_Pad1.30x1.75mm_HandSolder, B.Cu at (141.2, 66.5)
- added R3: 10k, Resistor_SMD:R_1206_3216Metric_Pad1.30x1.75mm_HandSolder, B.Cu at (141.2, 64.2)
- added R4: 10k, Resistor_SMD:R_1206_3216Metric_Pad1.30x1.75mm_HandSolder, B.Cu at (157.1, 60.4)
- added R5: 220, Resistor_SMD:R_1206_3216Metric_Pad1.30x1.75mm_HandSolder, B.Cu at (157.1, 62.7)
- added R6: 4.7k, Resistor_SMD:R_1206_3216Metric_Pad1.30x1.75mm_HandSolder, B.Cu at (182.7, 125.6)
- added R7: 4.7k, Resistor_SMD:R_1206_3216Metric_Pad1.30x1.75mm_HandSolder, B.Cu at (182.8, 105.8)
- added R8: 4.7k, Resistor_SMD:R_1206_3216Metric_Pad1.30x1.75mm_HandSolder, B.Cu at (182.9, 86.1)
- added R9: 4.7k, Resistor_SMD:R_1206_3216Metric_Pad1.30x1.75mm_HandSolder, B.Cu at (182.8, 66.6)
- added U10: AP2127K-1.8, Package_TO_SOT_SMD:SOT-23-5, B.Cu at (146.6, 91.4)
- added U2: MQ-x, Sensor:MQ-6, F.Cu at (182.6, 116.0)
- added U3: MQ-x, Sensor:MQ-6, F.Cu at (182.6, 96.2)
- added U4: MQ-x, Sensor:MQ-6, F.Cu at (182.8, 76.6)
- added U5: MQ-x, Sensor:MQ-6, F.Cu at (182.8, 56.9)
- added U6: BME280, Package_LGA:Bosch_LGA-8_2.5x2.5mm_P0.65mm_ClockwisePinNumbering, F.Cu at (179.3, 109.4)
- added U7: ENS160-BGLM, KML-Custom:XDCR_ENS160-BGLM, F.Cu at (178.3, 89.6)
- added U8: TXB0104D, Package_SO:SOIC-14_3.9x8.7mm_P1.27mm, B.Cu at (151.4, 53.8)
- added U9: AP2112K-3.3, Package_TO_SOT_SMD:SOT-23-5, B.Cu at (140.3, 52.4)
Connections:
- A1 pad 10: unconnected-(A1-D7-Pad10) -> /alarm
- A1 pad 11: unconnected-(A1-D8-Pad11) -> /heat_sw
- A1 pad 12: unconnected-(A1-D9-Pad12) -> /CD
- A1 pad 13: unconnected-(A1-D10-Pad13) -> /SS
- A1 pad 14: unconnected-(A1-D11-Pad14) -> /DI
- A1 pad 15: unconnected-(A1-D12-Pad15) -> /DO
- A1 pad 16: unconnected-(A1-D13-Pad16) -> /CLK
- A1 pad 17: unconnected-(A1-3V3-Pad17) -> +3V3
- A1 pad 19: unconnected-(A1-A0-Pad19) -> /GS4
- A1 pad 20: unconnected-(A1-A1-Pad20) -> /GS3
- A1 pad 21: unconnected-(A1-A2-Pad21) -> /GS2
- A1 pad 22: unconnected-(A1-A3-Pad22) -> /GS1
- A1 pad 25: unconnected-(A1-A6-Pad25) -> /Soft_CLK
- A1 pad 26: unconnected-(A1-A7-Pad26) -> /Soft_DAT
- A1 pad 9: unconnected-(A1-D6-Pad9) -> /CS
Routing:
- net +5V: track 108.9 -> 345.2 mm, vias 1 -> 3
- net /DI: track 0.00 -> 132.2 mm
- net /DO: track 0.00 -> 132.1 mm, vias 0 -> 2
- net /CLK: track 0.00 -> 125.0 mm, vias 0 -> 2
- net +3V3: track 0.00 -> 119.6 mm, vias 0 -> 3
- net /SS: track 0.00 -> 110.7 mm
- net /GS4: track 0.00 -> 106.1 mm, vias 0 -> 1
- net /alarm: track 0.00 -> 85.4 mm, vias 0 -> 1
- net /GS3: track 0.00 -> 85.3 mm, vias 0 -> 1
- net /heat_sw: track 0.00 -> 81.9 mm, vias 0 -> 4
- net /CD: track 0.00 -> 79.9 mm, vias 0 -> 2
- net /CS: track 0.00 -> 75.4 mm, vias 0 -> 2
- net GND: track 19.6 -> 89.4 mm, vias 14 -> 23
- net /GS2: track 0.00 -> 64.6 mm, vias 0 -> 1
- net +1V8: track 0.00 -> 54.0 mm, vias 0 -> 1
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