File: hardware/BREAD_Slice.kicad_pcb (KiCad board)
At the start: 2 copper layers, 70 x 100 mm, 69 parts, among them IC1 DS3234S#, J1 I2C_01x04, J2 Conn_01x10_Female, J3 MicroSD_502570-0893, K1 G5Q-1, Q1 IRLZ34N, Q2 IRLZ34N, U10 AP2127K-1.8, U2 MQ-x, U3 MQ-x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

Commit message: JLCPCB order rev-A
Parts:
- added G***: LOGO, LOGO, F.Cu at (168.8, 110.2)
Other:
- board text added: "BREAD Slice Industrial Air- Quality Monitor (SLC_IAQM) Cam K Brooks rev.A [09-2024]"
- board text removed: "BREAD Slice Template SLC_TEMP <version> <year>"
