File: hardware/BREAD_Slice.kicad_pcb (KiCad board)
At the start: 2 copper layers, 70 x 100 mm, 70 parts, among them IC1 DS3234S#, J1 I2C_01x04, J2 Conn_01x10_Female, J3 MicroSD_502570-0893, K1 G5Q-1, Q1 IRLZ34N, Q2 IRLZ34N, U10 AP2127K-1.8, U2 MQ-x, U3 MQ-x, U4 MQ-x, U5 MQ-x, U6 BME280, U7 ENS160-BGLM, U8 TXB0104D, U9 AP2112K-3.3

Commit message: fix(hw): re-point stale library nicknames
These parts exist in KiCad-Master-Lib; the boards referenced libraries that no
longer exist (kml-custom, KML-Custom, and SparkFun libraries that never
contained the part) or names the library has since changed.

KiCad embeds footprint geometry in the .kicad_pcb, so the boards rendered and
fabricated correctly and the rot stayed invisible -- it only surfaces on
update-from-library, or when a generator tries to resolve a nickname.

Nickname/name only. No geometry is changed:

  KML-Custom:H178CAD_P2.54mm_RightAngle_LED -> KMLib_Connectors:H178CAD_P2.54mm_RightAngle_LED
  KML-Custom:SOIC127P1032X265-20N -> KMLib_IC_SMD:SOIC127P1032X265-20N
  KML-Custom:Thermal Pad -> KMLib_Mounting:Thermal_Pad
  KML-Custom:XDCR_ENS160-BGLM -> KMLib_IC_SMD:XDCR_ENS160-BGLM
  SparkFun-DiscreteSemi:AP63205 -> KMLib_IC_Power:AP63205WU-7_Buck_Regulator
  SparkFun-LED:WS2812-5050-4PIN -> KMLib_IC_SMD:WS2812-5050-4PIN
  kml-custom:DS3234S# -> KMLib_Sensors:DS3234S_RTC
  kml-custom:ENS160-BGLM -> KMLib_Sensors:ENS160-BGLM_Air_Quality
  kml-custom:MicroSD_502570-0893 -> KMLib_Connectors:502570-0893_MicroSD_Molex

Only references that failed to resolve were touched. Generic parts (<=4 pins)
and KiCad *-rescue libraries are deliberately excluded: fingerprint matching
cannot distinguish a 2-pin resistor from a 2-pin capacitor, so those are being
done by hand.
Parts:
- D1: footprint SparkFun-LED:WS2812-5050-4PIN -> KMLib_IC_SMD:WS2812-5050-4PIN
- D2: footprint KML-Custom:H178CAD_P2.54mm_RightAngle_LED -> KMLib_Connectors:H178CAD_P2.54mm_RightAngle_LED
- HS1: footprint KML-Custom:Thermal Pad -> KMLib_Mounting:Thermal_Pad
- IC1: footprint KML-Custom:SOIC127P1032X265-20N -> KMLib_IC_SMD:SOIC127P1032X265-20N
- U7: footprint KML-Custom:XDCR_ENS160-BGLM -> KMLib_IC_SMD:XDCR_ENS160-BGLM
Changed lines of the file:
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@@
 		(embedded_fonts no)
 	)
-	(footprint "KML-Custom:Thermal Pad"
+	(footprint "KMLib_Mounting:Thermal_Pad"
 		(layer "F.Cu")
 		(at 131.35 121.355)
@@
 		)
 	)
-	(footprint "SparkFun-LED:WS2812-5050-4PIN"
+	(footprint "KMLib_IC_SMD:WS2812-5050-4PIN"
 		(locked yes)
 		(layer "F.Cu")
@@
 		(embedded_fonts no)
 	)
-	(footprint "KML-Custom:XDCR_ENS160-BGLM"
+	(footprint "KMLib_IC_SMD:XDCR_ENS160-BGLM"
 		(layer "F.Cu")
 		(at 178.315076 89.6 45)
@@
 		)
 	)
-	(footprint "KML-Custom:H178CAD_P2.54mm_RightAngle_LED"
+	(footprint "KMLib_Connectors:H178CAD_P2.54mm_RightAngle_LED"
 		(layer "F.Cu")
 		(at 135.52 45.58 90)
@@
 		)
 	)
-	(footprint "KML-Custom:SOIC127P1032X265-20N"
+	(footprint "KMLib_IC_SMD:SOIC127P1032X265-20N"
 		(layer "B.Cu")
 		(at 168.425 54.788 -90)
