File: hardware/mq_gas_sensor.kicad_sch (KiCad schematic)
At the start: 2 parts, among them U4 MQ-x

Commit message: completed schematic
Parts:
- renumbered R3 to R8, U4 to U2
Other:
- moved on the sheet: R8, U2

Commit message: organized schem and updated readme
Parts:
- renumbered R8 to R4
Changed lines of the file:
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@@
 		(dnp no)
 		(fields_autoplaced yes)
-		(property "Reference" "R8"
+		(property "Reference" "R4"
 			(at 139.7 95.2499 0)
 			(effects
@@
 			(project "BREAD_Slice"
 				(path "/66043bca-a260-4915-9fce-8a51d324c687/268aacf0-fff4-4b55-82e7-cfe6b1e82ea8"
-					(reference "R8")
+					(reference "R4")
 					(unit 1)
 				)
 				(path "/66043bca-a260-4915-9fce-8a51d324c687/cab85a36-8baf-4341-ae39-bf466ad69f78"
-					(reference "R9")
+					(reference "R5")
 					(unit 1)
 				)
 				(path "/66043bca-a260-4915-9fce-8a51d324c687/fe6fce18-dda6-45f5-ac36-63e733626505"
-					(reference "R10")
+					(reference "R6")
 					(unit 1)
 				)
 				(path "/66043bca-a260-4915-9fce-8a51d324c687/134c4f80-1fbc-4764-a894-22f604c6d155"
-					(reference "R7")
+					(reference "R3")
 					(unit 1)
 				)

Commit message: completed board
Parts:
- R7: renamed from R4; footprint (none) -> Resistor_SMD:R_1206_3216Metric_Pad1.30x1.75mm_HandSolder
Changed lines of the file:
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@@
 		(dnp no)
 		(fields_autoplaced yes)
-		(property "Reference" "R4"
+		(property "Reference" "R7"
 			(at 139.7 95.2499 0)
 			(effects
@@
 			)
 		)
-		(property "Footprint" ""
+		(property "Footprint" "Resistor_SMD:R_1206_3216Metric_Pad1.30x1.75mm_HandSolder"
 			(at 144.018 96.52 90)
 			(effects
@@
 			(project "BREAD_Slice"
 				(path "/66043bca-a260-4915-9fce-8a51d324c687/268aacf0-fff4-4b55-82e7-cfe6b1e82ea8"
-					(reference "R4")
+					(reference "R7")
 					(unit 1)
 				)
 				(path "/66043bca-a260-4915-9fce-8a51d324c687/cab85a36-8baf-4341-ae39-bf466ad69f78"
-					(reference "R5")
+					(reference "R8")
 					(unit 1)
 				)
 				(path "/66043bca-a260-4915-9fce-8a51d324c687/fe6fce18-dda6-45f5-ac36-63e733626505"
+					(reference "R9")
+					(unit 1)
+				)
+				(path "/66043bca-a260-4915-9fce-8a51d324c687/134c4f80-1fbc-4764-a894-22f604c6d155"
 					(reference "R6")
 					(unit 1)
 				)
-				(path "/66043bca-a260-4915-9fce-8a51d324c687/134c4f80-1fbc-4764-a894-22f604c6d155"
-					(reference "R3")
-					(unit 1)
-				)

Commit message: checked output for order
Parts:
- renumbered R7 to R6
Changed lines of the file:
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@@
 		(dnp no)
 		(fields_autoplaced yes)
-		(property "Reference" "R7"
+		(property "Reference" "R6"
 			(at 139.7 95.2499 0)
 			(effects
