File: hardware/BREAD_Slice.kicad_sch (KiCad schematic)
At the start: 29 parts, among them J1 I2C_01x04, J2 Conn_01x10_Female, K1 G5Q-1, Q1 IRLZ34N, Q2 IRLZ34N, U1 AP63205WU-7

Commit message: fix(hw): re-point stale library nicknames
These parts exist in KiCad-Master-Lib; the boards referenced libraries that no
longer exist (kml-custom, KML-Custom, and SparkFun libraries that never
contained the part) or names the library has since changed.

KiCad embeds footprint geometry in the .kicad_pcb, so the boards rendered and
fabricated correctly and the rot stayed invisible -- it only surfaces on
update-from-library, or when a generator tries to resolve a nickname.

Nickname/name only. No geometry is changed:

  KML-Custom:H178CAD_P2.54mm_RightAngle_LED -> KMLib_Connectors:H178CAD_P2.54mm_RightAngle_LED
  KML-Custom:SOIC127P1032X265-20N -> KMLib_IC_SMD:SOIC127P1032X265-20N
  KML-Custom:Thermal Pad -> KMLib_Mounting:Thermal_Pad
  KML-Custom:XDCR_ENS160-BGLM -> KMLib_IC_SMD:XDCR_ENS160-BGLM
  SparkFun-DiscreteSemi:AP63205 -> KMLib_IC_Power:AP63205WU-7_Buck_Regulator
  SparkFun-LED:WS2812-5050-4PIN -> KMLib_IC_SMD:WS2812-5050-4PIN
  kml-custom:DS3234S# -> KMLib_Sensors:DS3234S_RTC
  kml-custom:ENS160-BGLM -> KMLib_Sensors:ENS160-BGLM_Air_Quality
  kml-custom:MicroSD_502570-0893 -> KMLib_Connectors:502570-0893_MicroSD_Molex

Only references that failed to resolve were touched. Generic parts (<=4 pins)
and KiCad *-rescue libraries are deliberately excluded: fingerprint matching
cannot distinguish a 2-pin resistor from a 2-pin capacitor, so those are being
done by hand.
Parts:
- D1: footprint SparkFun-LED:WS2812-5050-4PIN -> KMLib_IC_SMD:WS2812-5050-4PIN
- D2: footprint KML-Custom:H178CAD_P2.54mm_RightAngle_LED -> KMLib_Connectors:H178CAD_P2.54mm_RightAngle_LED
- HS1: footprint KML-Custom:Thermal Pad -> KMLib_Mounting:Thermal_Pad
- U1: symbol SparkFun-DiscreteSemi:AP63205 -> KMLib_IC_Power:AP63205WU-7_Buck_Regulator
Changed lines of the file:
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@@
 	)
 	(symbol
-		(lib_id "SparkFun-DiscreteSemi:AP63205")
+		(lib_id "KMLib_IC_Power:AP63205WU-7_Buck_Regulator")
 		(at 31.75 96.52 0)
 		(unit 1)
@@
 			)
 		)
-		(property "Footprint" "KML-Custom:Thermal Pad"
+		(property "Footprint" "KMLib_Mounting:Thermal_Pad"
 			(at 45.72 112.0648 0)
 			(hide yes)
@@
 			)
 		)
-		(property "Footprint" "KML-Custom:H178CAD_P2.54mm_RightAngle_LED"
+		(property "Footprint" "KMLib_Connectors:H178CAD_P2.54mm_RightAngle_LED"
 			(at 130.81 167.64 0)
 			(hide yes)
@@
 			)
 		)
-		(property "Footprint" "SparkFun-LED:WS2812-5050-4PIN"
+		(property "Footprint" "KMLib_IC_SMD:WS2812-5050-4PIN"
 			(at 49.53 76.2 0)
 			(hide yes)
